Commit message: Port RoARM-M2-S to ROS 2 Jazzy
- Fix ikfast plugin: update .h headers to .hpp for Jazzy compatibility
- Remove ament_export_targets from ikfast CMakeLists to prevent LD_LIBRARY_PATH pollution
- Fix ros2_controllers.yaml: add open_loop_control and allow_integration_in_goal_trajectories
- Fix joint_limits.yaml: enable has_acceleration_limits for all joints
- Fix moveit_controllers.yaml: correct gripper action_ns to follow_joint_trajectory
- Remove deleted moveit_servo (bundled Humble version, use system Jazzy package instead)
- Remove roarm_moveit_cmd (incompatible, needs separate porting)

File: src/roarm_main/roarm_description/urdf/roarm_description.urdf (robot description, URDF)
Before this commit: robot roarm_description, 6 links, 5 joints
Joints:
- joint base_link_to_link1: limit lower=-3.1416 upper=3.1416 effort=0 velocity=0 -> lower=-3.1416 upper=3.1416 effort=10.0 velocity=1.0
- joint link1_to_link2: limit lower=-1.5708 upper=1.5708 effort=0 velocity=0 -> lower=-1.5708 upper=1.5708 effort=10.0 velocity=1.0
- joint link2_to_link3: limit lower=-1 upper=3.1416 effort=0 velocity=0 -> lower=-1 upper=3.1416 effort=10.0 velocity=1.0
- joint link3_to_gripper_link: limit lower=0 upper=1.5 effort=0 velocity=0 -> lower=0 upper=1.5 effort=10.0 velocity=1.0
- joint link3_to_hand_tcp: axis 0 0 0 -> (none)

File: src/roarm_main/roarm_moveit/config/roarm_description.ros2_control.xacro (robot description, xacro)
@@ -2,5 +2,5 @@
 <robot xmlns:xacro="http://www.ros.org/wiki/xacro">
     <xacro:macro name="roarm_description_ros2_control" params="name initial_positions_file">
-        <xacro:property name="initial_positions" value="${load_yaml(initial_positions_file)['initial_positions']}"/>
+        <xacro:property name="initial_positions" value="${xacro.load_yaml(initial_positions_file)['initial_positions']}"/>
         <ros2_control name="${name}" type="system">
             <hardware>
@@ -13,5 +13,7 @@
                   <param name="initial_value">${initial_positions['base_link_to_link1']}</param>
                 </state_interface>
-                <state_interface name="velocity"/>
+                <state_interface name="velocity">
+                    <param name="initial_value">0.0</param>
+                </state_interface>
             </joint>
             <joint name="link1_to_link2">
@@ -20,5 +22,7 @@
                   <param name="initial_value">${initial_positions['link1_to_link2']}</param>
                 </state_interface>
-                <state_interface name="velocity"/>
+                <state_interface name="velocity">
+                    <param name="initial_value">0.0</param>
+                </state_interface>
             </joint>
             <joint name="link2_to_link3">
@@ -27,5 +31,7 @@
                   <param name="initial_value">${initial_positions['link2_to_link3']}</param>
                 </state_interface>
-                <state_interface name="velocity"/>
+                <state_interface name="velocity">
+                    <param name="initial_value">0.0</param>
+                </state_interface>
             </joint>
             <joint name="link3_to_gripper_link">
@@ -34,5 +40,7 @@
                   <param name="initial_value">${initial_positions['link3_to_gripper_link']}</param>
                 </state_interface>
-                <state_interface name="velocity"/>
+                <state_interface name="velocity">
+                    <param name="initial_value">0.0</param>
+                </state_interface>
             </joint>
         </ros2_control>
