Commit message: updated the roarm_description.urdf

File: src/roarm_main/roarm_description/urdf/roarm_description.urdf (robot description, URDF)
Before this commit: robot roarm_description, 6 links, 5 joints
Joints:
- joint link3_to_gripper_link: limit lower=0 upper=1.5 effort=10.0 velocity=1.0 -> lower=-1.2 upper=3 effort=10.0 velocity=1.0
